File: CPEG298_SMART-MFC/CPEG298_SMART-MFC.kicad_pcb (KiCad board)
At the start: 2 copper layers, 68.6 x 53.3 mm, 8 parts, among them J1 Power, J2 Digital/PWM, J3 Analog, J4 Digital/PWM

Commit message: Lab4_Complete
Parts:
- added C1: C_Polarized_US, Capacitor_THT:CP_Radial_D6.3mm_P2.50mm, F.Cu at (138.1, 87.3)
- added R1: 1000, Resistor_THT:R_Axial_DIN0207_L6.3mm_D2.5mm_P10.16mm_Horizontal, F.Cu at (138.1, 62.9)
- added R2: 2000, Resistor_THT:R_Axial_DIN0207_L6.3mm_D2.5mm_P10.16mm_Horizontal, F.Cu at (138.1, 67.0)
- added U1: ESP8266-01/ESP-01, ESP8266-01_ESP-01:XCVR_ESP8266-01_ESP-01, F.Cu at (166.7, 63.2)
Routing:
- net /SDA/A4: track 0.00 -> 88.2 mm
- net /SCL/A5: track 0.00 -> 81.7 mm
- net /*10: track 0.00 -> 23.5 mm
- net +5V: track 0.00 -> 10.2 mm
- added copper zone on B.Cu, net GND

Commit message: Lab5
-Added Grove Connectors
-Rewiring
-3D STEP Files
-New Libraries
*SEEED, Digikey
Parts:
- added J5: Soil_Moisture_Sensor, OPL_Connector:HW4-2.0, F.Cu at (154.2, 86.8)
- added J6: Temperature_Sensor, OPL_Connector:HW4-2.0, F.Cu at (161.0, 86.8)
- added J7: Light_Sensor, OPL_Connector:HW4-2.0, F.Cu at (146.6, 86.8)
- moved R1 4.38 mm to (135.6, 59.4), turned to -90 degrees
- moved R2 3.59 mm to (140.6, 69.5), turned to 90 degrees
- turned C1 to 180 degrees
Connections:
- J3 pad 5: /SDA/A4 -> /A4
- J3 pad 6: /SCL/A5 -> /A5
Routing:
- net /SDA/A4: track 88.2 -> 0.19 mm
- net /SCL/A5: track 81.7 -> 0.00 mm
- net +5V: track 10.2 -> 36.5 mm
- net Net-(U1-RXD): track 0.00 -> 23.9 mm
- net /*11: track 0.00 -> 10.8 mm
- net /A4: track 0.00 -> 10.4 mm
- net /A0: track 0.00 -> 9.38 mm
- net /A5: track 0.00 -> 8.67 mm
- net /A2: track 0.00 -> 8.33 mm
- net /*10: track 23.5 -> 25.6 mm
