File: CPEG298_SMART-MFC/_autosave-CPEG298_SMART-MFC.kicad_pcb (KiCad board)
At the start: 2 copper layers, 68.6 x 53.3 mm, 19 parts, among them J1 Power, J2 Digital/PWM, J3 Analog, J4 Digital/PWM, J5 Soil_Moisture_Sensor, J6 Temperature_Sensor, J7 Light_Sensor, J8 LCD, U1 ESP8266-01/ESP-01

Commit message: KiCad Components and Software
Parts:
- added G***: LOGO, LOGO, F.Cu at (115.2, 69.5)
