File: CPEG298_SMART-MFC/_autosave-CPEG298_SMART-MFC.kicad_pcb (KiCad board)
At the start: 2 copper layers, 68.6 x 53.3 mm, 21 parts, among them J1 Power, J2 Digital/PWM, J3 Analog, J4 Digital/PWM, J5 Soil, J6 Temp., J7 Light, J8 LCD, U1 ESP8266-01/ESP-01

Commit message: KiCad & Code
-Labeling on PCB
-Preparing code for millivolt reader
Parts:
- removed the G*** at (135.6, 72.1)
- J5: value Soil -> Soil_Moisture_Sensor
- J6: value Temp. -> Temperature_Sensor
- J7: value Light -> Light_Sensor
Other:
- board text removed: "3V3"
- board text removed: "5V"
- board text removed: "GND"
- board text removed: "MM"
- board text removed: "RT"
- board text removed: "VCC"
