File: CPEG298_SMART-MFC/_autosave-CPEG298_SMART-MFC.kicad_pcb (KiCad board)
At the start: 2 copper layers, 68.6 x 53.3 mm, 25 parts, among them J1 Power, J2 Digital/PWM, J3 Analog, J4 Digital/PWM, J5 Soil, J6 Temp, J7 Light, U1 ESP8266-01

Commit message: Submission for Review
Parts:
- removed D2: Temperature, LED_THT:LED_D5.0mm
- removed the G*** at (162.4, 76.0)
- removed the G*** at (135.6, 72.1)
- removed R4, R5, R6: 1000, Resistor_THT:R_Axial_DIN0207_L6.3mm_D2.5mm_P10.16mm_Horizontal
- added J8: LCD, OPL_Connector:HW4-2.0, F.Cu at (184.2, 79.8)
- C2: value C -> C_Polarized_US
- D1: value Soil Moisture -> Soil Moisture Threshold
- J5: value Soil -> Soil_Moisture_Sensor
- J6: value Temp -> Temperature_Sensor
- J7: value Light -> Light_Sensor
- R3: value 1000 -> R
- U1: value ESP8266-01 -> ESP8266-01/ESP-01
- moved D1 2.54 mm to (107.6, 51.7), turned to 180 degrees
- moved G*** 2.54 mm to (115.2, 69.5)
Connections:
- D1 pad 1: GND -> Net-(D1-K)
- D1 pad 2: Net-(D1-A) -> GND
- J1 pad 1: /InputMillivolt -> unconnected-(J1-Pin_1-Pad1)
- J1 pad 4: +3.3V -> +3V3
- J6 pad 1: /SCL/A5 -> /A5
- J6 pad 2: /SDA/A4 -> /A4
- R3 pad 2: Net-(D1-A) -> Net-(D1-K)
Routing:
- net /SCL/A5: track 76.0 -> 0.00 mm
- net /SDA/A4: track 72.8 -> 0.19 mm
- net Net-(D2-A): track 60.5 -> 0.00 mm
- net Net-(D1-K): track 0.00 -> 37.7 mm
- net Net-(D1-A): track 37.7 -> 0.00 mm
- net /InputMillivolt: track 28.6 -> 0.00 mm
- net /A1: track 25.0 -> 0.00 mm
- net +3.3V: track 64.7 -> 52.5 mm
- net /*6: track 11.2 -> 0.00 mm
- net /A4: track 0.00 -> 10.4 mm
- net /A5: track 0.00 -> 8.67 mm
- net Net-(U1-RXD): track 26.0 -> 23.9 mm
Other:
- board text added: "SMART MFC IoT Rev. A 3/13/2023 Michael Earley"
- board text removed: "0"
- board text removed: "3V3"
- board text removed: "5V"
- board text removed: "A0"
- board text removed: "GND"
- board text removed: "MM"
- board text removed: "RT"
- board text removed: "SCL SDA"
- board text removed: "SMART MFC IoT Rev. A 3/17/2023 Michael Earley"
- board text removed: "Too High!"
- board text removed: "VCC"
- board text removed: "a"
