File: CPEG298_SMART-MFC/CPEG298_SMART-MFC.kicad_sch (KiCad schematic)
At the start: 4 parts, among them J1 Power, J2 Digital/PWM, J3 Analog, J4 Digital/PWM

Commit message: Submission for Review
Parts:
- added C1: C_Polarized_US, Capacitor_THT:CP_Radial_D6.3mm_P2.50mm, symbol Device:C_Polarized_US
- added C2: C, Capacitor_THT:CP_Radial_D6.3mm_P2.50mm, symbol Device:C_Polarized_US
- added D1: Soil Moisture, LED_THT:LED_D5.0mm, symbol Device:LED
- added D2: Temperature, LED_THT:LED_D5.0mm, symbol Device:LED
- added J5: Soil, OPL_Connector:HW4-2.0, symbol OPL_Connector:GROVE-CONNECTOR-DIP_4P-2.0_
- added J6: Temp, OPL_Connector:HW4-2.0, symbol OPL_Connector:GROVE-CONNECTOR-DIP_4P-2.0_
- added J7: Light, OPL_Connector:HW4-2.0, symbol OPL_Connector:GROVE-CONNECTOR-DIP_4P-2.0_
- added R1, R3, R4, R5, R6: 1000, Resistor_THT:R_Axial_DIN0207_L6.3mm_D2.5mm_P10.16mm_Horizontal, symbol Device:R_US
- added R2: 2000, Resistor_THT:R_Axial_DIN0207_L6.3mm_D2.5mm_P10.16mm_Horizontal, symbol Device:R_US
- added U1: ESP8266-01, ESP8266-01_ESP-01:XCVR_ESP8266-01_ESP-01, symbol ESP8266-01_ESP-01:ESP8266-01/ESP-01
Connections:
- net *10: now also U1.5 (TXD)
- net *11: now also R1.1
- net *6: now also R6.1
- net +5V: now also C1.1, J5.3, J6.3, J7.3
- net 7: now also R3.1
- net A0: now also J7.1
- net A1: now also R4.2, R5.1
- net A2: now also J5.1
- net GND: now also C1.2, C2.2, D1.1 (K), D2.1 (K), J5.4, J6.4, J7.4, R2.2, R5.2, U1.1 (GND)
- net SCL/A5: now also J6.1; no longer J3.6 (Pin_6)
- net SDA/A4: now also J6.2; no longer J3.5 (Pin_5)
- net InputMillivolt: now reaches J1.1 (Pin_1)
- net InputMillivolt: now also R4.1
- new net: D2.2 (A), R6.2
- new net: R1.2, R2.1, U1.4 (RXD)
- new net: D1.2 (A), R3.2
- new net +3.3V: C2.1, U1.6 (EN), U1.8 (VCC)
- new net A4: J3.5 (Pin_5)
- new net A5: J3.6 (Pin_6)
- no-connect marks 1 -> 21
